Commit message: update task

File: assets/urdf/objects/cube_multicolor_allegro.urdf (robot description, URDF)
Before this commit: robot object, 1 links, 0 joints
Links:
- link object: geometry collision box size=0.05 0.05 0.05; visual mesh filename=meshes/cube_multicolor.obj scale=.05 .05 .05

Commit message: update cube

File: assets/urdf/objects/cube_multicolor_allegro.urdf (robot description, URDF)
Before this commit: robot object, 1 links, 0 joints
Links:
- link object: geometry collision box size=0.06 0.06 0.06; visual mesh filename=meshes/cube_multicolor.obj scale=.06 .06 .06
